Commit message: add cab to urdf

File: ros/lazerbot_tf/src/lazerbot_tf.urdf (robot description, URDF)
Before this commit: robot lazerbot, 5 links, 4 joints
Links:
- added link bed_link; visual box size=0.28 0.26 0.06
- added link cab_link; visual box size=0.227 0.244 0.27
- link base_link: geometry visual box size=0.35 0.175 0.041
Joints:
- added joint bed_joint: type fixed, parent base_link, child bed_link, origin xyz=-0.065 0 0.051
- added joint cab_joint: type fixed, parent base_link, child cab_link, origin xyz=0.189 0 0.155
- joint wheel_joint_bl: origin xyz=0.105 -0.099 -0.008 rpy=0 0 0 -> xyz=-0.105 -0.099 -0.008 rpy=0 0 0
- joint wheel_joint_br: origin xyz=0.105 0.099 -0.008 rpy=0 0 0 -> xyz=-0.105 0.099 -0.008 rpy=0 0 0
- joint wheel_joint_fl: origin xyz=-0.105 -0.099 -0.008 rpy=0 0 0 -> xyz=0.105 -0.099 -0.008 rpy=0 0 0
- joint wheel_joint_fr: origin xyz=-0.105 0.099 -0.008 rpy=0 0 0 -> xyz=0.105 0.099 -0.008 rpy=0 0 0
